Commit message: Generate resource URDFs (planning, spherized, viz) + ship meshes
Mirrors autolife_planning/resources/robot/autolife/ layout:

  bimanual_franka_planning/resources/robot/bimanual_fr3/
    bimanual_fr3.urdf            # planning URDF (mesh collision)
    bimanual_fr3_spherized.urdf  # FK-gen input (sphere collision only)
    bimanual_fr3_viz.urdf        # PyBullet GUI (visual only)
    bimanual_fr3.srdf            # collision-pair filters
    meshes/                      # collision .stl
    viz_meshes/                  # high-poly visual .dae

URDFs reference meshes via package://meshes/... — the PyBullet env's
package resolver walks up from the URDF directory until it finds a
matching folder, so ROS isn't required.

Mesh references are unified to plain "package://meshes/..." across
both the assets/ source URDF and the package resource URDFs.

File: bimanual_franka_planning/resources/robot/bimanual_fr3/bimanual_fr3_viz.urdf (robot description, URDF)
Before this commit: robot bimanual_fr3, 28 links, 27 joints
Links:
- link fr3_left_hand: geometry visual mesh filename=package://meshes/robot_ee/franka_hand_white/visual/hand.dae
- link fr3_left_leftfinger: geometry visual mesh filename=package://meshes/robot_ee/franka_hand_white/visual/finger.d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
- link fr3_left_link0: geometry visual mesh filename=package://meshes/robot_arms/fr3/visual/link0.dae
- link fr3_left_link1: geometry visual mesh filename=package://meshes/robot_arms/fr3/visual/link1.dae
- link fr3_left_link2: geometry visual mesh filename=package://meshes/robot_arms/fr3/visual/link2.dae
- link fr3_left_link3: geometry visual mesh filename=package://meshes/robot_arms/fr3/visual/link3.dae
- link fr3_left_link4: geometry visual mesh filename=package://meshes/robot_arms/fr3/visual/link4.dae
- link fr3_left_link5: geometry visual mesh filename=package://meshes/robot_arms/fr3/visual/link5.dae
- link fr3_left_link6: geometry visual mesh filename=package://meshes/robot_arms/fr3/visual/link6.dae
- link fr3_left_link7: geometry visual mesh filename=package://meshes/robot_arms/fr3/visual/link7.dae
- link fr3_left_rightfinger: geometry visual mesh filename=package://meshes/robot_ee/franka_hand_white/visual/finger.d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
- link fr3_right_hand: geometry visual mesh filename=package://meshes/robot_ee/franka_hand_white/visual/hand.dae
- link fr3_right_leftfinger: geometry visual mesh filename=package://meshes/robot_ee/franka_hand_white/visual/finger.d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
- link fr3_right_link0: geometry visual mesh filename=package://meshes/robot_arms/fr3/visual/link0.dae
- link fr3_right_link1: geometry visual mesh filename=package://meshes/robot_arms/fr3/visual/link1.dae
- link fr3_right_link2: geometry visual mesh filename=package://meshes/robot_arms/fr3/visual/link2.dae
- link fr3_right_link3: geometry visual mesh filename=package://meshes/robot_arms/fr3/visual/link3.dae
- link fr3_right_link4: geometry visual mesh filename=package://meshes/robot_arms/fr3/visual/link4.dae
- link fr3_right_link5: geometry visual mesh filename=package://meshes/robot_arms/fr3/visual/link5.dae
- link fr3_right_link6: geometry visual mesh filename=package://meshes/robot_arms/fr3/visual/link6.dae
- link fr3_right_link7: geometry visual mesh filename=package://meshes/robot_arms/fr3/visual/link7.dae
- link fr3_right_rightfinger: geometry visual mesh filename=package://meshes/robot_ee/franka_hand_white/visual/finger.d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
