Commit message: Add relative-base DOF design + Python types + robot description
Frame design:
  ``world`` is co-located with ``fr3_left_link0`` so deployment
  calibration is purely the relative pose of the right arm. The
  right-arm base attaches to world through a 3-DOF planar chain
  (relative_base_x/y/yaw); pin those via base_config to plan single-
  arm motion at a known cell layout, or leave them active for layout
  search.

Joint order in the 17-DOF state vector (matches cricket FK header):
  [0:3]    relative_base   (x, y, yaw)
  [3:10]   right arm       (fr3_right_joint1..7)
  [10:17]  left arm        (fr3_left_joint1..7)

Spherized URDF now keeps both <sphere> collisions AND visual mesh
geometry, so a viewer can render the collision proxy alongside the
high-poly model — useful for sanity-checking spherization.

SRDF inherits per-arm exclusions from the cricket fr3.srdf without
adding any cross-arm exclusions, so the two arms collision-check
against each other.

Also adds:
  - bimanual_franka_planning/types/* (verbatim types module)
  - bimanual_franka_planning/utils/rot_utils.py
  - bimanual_franka_planning.bimanual_franka — robot description
  - pyproject.toml + pixi.toml mirroring autolife's build config

File: assets/bimanual_fr3_description/urdf/bimanual_fr3.urdf (robot description, URDF)
Before this commit: robot bimanual_fr3, 28 links, 27 joints
Links:
- added link relative_base_x_link
- added link relative_base_y_link
Joints:
- removed joint world_to_fr3_right_base
- added joint relative_base_x: type prismatic, parent world, child relative_base_x_link, origin xyz=0.0 0.0 0.0 rpy=0.0 0.0 0.0, axis 1 0 0, limit lower=-1.5 upper=1.5 effort=100.0 velocity=0.5
- added joint relative_base_y: type prismatic, parent relative_base_x_link, child relative_base_y_link, origin xyz=0.0 0.0 0.0 rpy=0.0 0.0 0.0, axis 0 1 0, limit lower=-1.5 upper=1.5 effort=100.0 velocity=0.5
- added joint relative_base_yaw: type revolute, parent relative_base_y_link, child fr3_right_link0, origin xyz=0.0 0.0 0.0 rpy=0.0 0.0 0.0, axis 0 0 1, limit lower=-3.14159265 upper=3.14159265 effort=100.0 velocity=1.0
- joint world_to_camera: origin xyz=0.5 0.0 0.6 rpy=0.0 0.3 0.0 -> xyz=0.5 -0.4 0.6 rpy=0.0 0.3 0.0
- joint world_to_fr3_left_base: origin xyz=0.0 0.4 0.0 rpy=0.0 0.0 0.0 -> xyz=0 0 0 rpy=0 0 0

File: bimanual_franka_planning/resources/robot/bimanual_fr3/bimanual_fr3_spherized.urdf (robot description, URDF)
Before this commit: robot bimanual_fr3, 28 links, 27 joints
Links:
- added link relative_base_x_link
- added link relative_base_y_link
- link fr3_left_hand: geometry collision sphere radius=0.043995; collision sphere radius=0.044394
- link fr3_left_leftfinger: geometry collision sphere radius=0.00429; collision sphere radius=0.004564
- link fr3_left_link0: geometry collision sphere radius=0.093646; collision sphere radius=0.117857
- link fr3_left_link1: geometry collision sphere radius=0.063841; collision sphere radius=0.076596
- link fr3_left_link2: geometry collision sphere radius=0.062048; collision sphere radius=0.076816
- link fr3_left_link3: geometry collision sphere radius=0.062048; collision sphere radius=0.075019
- link fr3_left_link4: geometry collision sphere radius=0.055149; collision sphere radius=0.075361
- link fr3_left_link5: geometry collision sphere radius=0.037086; collision sphere radius=0.038546
- link fr3_left_link6: geometry collision sphere radius=0.076831; collision sphere radius=0.082713
- link fr3_left_link7: geometry collision sphere radius=0.042595; collision sphere radius=0.054563
- link fr3_left_rightfinger: geometry collision sphere radius=0.00429; collision sphere radius=0.004564
- link fr3_right_hand: geometry collision sphere radius=0.043995; collision sphere radius=0.044394
- link fr3_right_leftfinger: geometry collision sphere radius=0.00429; collision sphere radius=0.004564
- link fr3_right_link0: geometry collision sphere radius=0.093646; collision sphere radius=0.117857
- link fr3_right_link1: geometry collision sphere radius=0.063841; collision sphere radius=0.076596
- link fr3_right_link2: geometry collision sphere radius=0.062048; collision sphere radius=0.076816
- link fr3_right_link3: geometry collision sphere radius=0.062048; collision sphere radius=0.075019
- link fr3_right_link4: geometry collision sphere radius=0.055149; collision sphere radius=0.075361
- link fr3_right_link5: geometry collision sphere radius=0.037086; collision sphere radius=0.038546
- link fr3_right_link6: geometry collision sphere radius=0.076831; collision sphere radius=0.082713
- link fr3_right_link7: geometry collision sphere radius=0.042595; collision sphere radius=0.054563
- link fr3_right_rightfinger: geometry collision sphere radius=0.00429; collision sphere radius=0.004564
Joints:
- removed joint world_to_fr3_right_base
- added joint relative_base_x: type prismatic, parent world, child relative_base_x_link, origin xyz=0.0 0.0 0.0 rpy=0.0 0.0 0.0, axis 1 0 0, limit lower=-1.5 upper=1.5 effort=100.0 velocity=0.5
- added joint relative_base_y: type prismatic, parent relative_base_x_link, child relative_base_y_link, origin xyz=0.0 0.0 0.0 rpy=0.0 0.0 0.0, axis 0 1 0, limit lower=-1.5 upper=1.5 effort=100.0 velocity=0.5
- added joint relative_base_yaw: type revolute, parent relative_base_y_link, child fr3_right_link0, origin xyz=0.0 0.0 0.0 rpy=0.0 0.0 0.0, axis 0 0 1, limit lower=-3.14159265 upper=3.14159265 effort=100.0 velocity=1.0
- joint world_to_camera: origin xyz=0.5 0.0 0.6 rpy=0.0 0.3 0.0 -> xyz=0.5 -0.4 0.6 rpy=0.0 0.3 0.0
- joint world_to_fr3_left_base: origin xyz=0.0 0.4 0.0 rpy=0.0 0.0 0.0 -> xyz=0 0 0 rpy=0 0 0

File: bimanual_franka_planning/resources/robot/bimanual_fr3/bimanual_fr3_viz.urdf (robot description, URDF)
Before this commit: robot bimanual_fr3, 28 links, 27 joints
Links:
- added link relative_base_x_link
- added link relative_base_y_link
Joints:
- removed joint world_to_fr3_right_base
- added joint relative_base_x: type prismatic, parent world, child relative_base_x_link, origin xyz=0.0 0.0 0.0 rpy=0.0 0.0 0.0, axis 1 0 0, limit lower=-1.5 upper=1.5 effort=100.0 velocity=0.5
- added joint relative_base_y: type prismatic, parent relative_base_x_link, child relative_base_y_link, origin xyz=0.0 0.0 0.0 rpy=0.0 0.0 0.0, axis 0 1 0, limit lower=-1.5 upper=1.5 effort=100.0 velocity=0.5
- added joint relative_base_yaw: type revolute, parent relative_base_y_link, child fr3_right_link0, origin xyz=0.0 0.0 0.0 rpy=0.0 0.0 0.0, axis 0 0 1, limit lower=-3.14159265 upper=3.14159265 effort=100.0 velocity=1.0
- joint world_to_camera: origin xyz=0.5 0.0 0.6 rpy=0.0 0.3 0.0 -> xyz=0.5 -0.4 0.6 rpy=0.0 0.3 0.0
- joint world_to_fr3_left_base: origin xyz=0.0 0.4 0.0 rpy=0.0 0.0 0.0 -> xyz=0 0 0 rpy=0 0 0
