Commit message: Add gripper as a planning DOF across all four FR3 variants
Each FR3 gripper now contributes its parallel-jaw fingers to the
configuration vector instead of being silently fixed in the URDF:

  • single_fr3 / single_fr3_soft  : 7 → 9 DOF (+ finger_joint1/2)
  • bimanual_fr3 / bimanual_fr3_soft : 17 → 21 DOF (+ 2 per arm)

URDF: ``fr3_*_finger_joint1`` becomes ``prismatic`` with travel
[0, 0.04] m; ``finger_joint2`` is declared as a ``<mimic>`` of joint1
so any consumer that honors mimic (Pinocchio, MuJoCo, PyBullet viz)
keeps the gripper symmetric automatically.  q=0 is fully closed,
q=0.04 is fully open with an 80 mm gap — matching the rigid Franka
semantics on both rigid and soft variants.

Cricket parses ``<mimic>`` but treats both finger joints as
independent in the FK output, so the planner exposes them as two
DOFs per gripper.  By convention callers should keep them equal;
the docstrings in each robot description module document this.

SRDF generation fix in ``tools/build_bimanual_urdf.py``: the bimanual
URDF prefixes link names with ``fr3_left_/fr3_right_``, but the
SRDF transformer only renamed ``fr3_link*`` and ``fr3_joint*``.
Once the fingers became prismatic (and therefore visible to the
collision checker as movable bodies) the un-prefixed
``disable_collisions`` rules for ``fr3_hand`` / ``fr3_leftfinger`` /
``fr3_rightfinger`` no longer matched any link, and HOME validated
as in collision.  Added explicit prefix substitutions for those
three link names.

New examples
  • examples/planning/gripper_motion.py — three idiomatic ways to
    drive the gripper through configuration space (whole-body plan,
    combined arm+gripper, gripper-only subgroup).
  • examples/planning/gripper_motion_vis.py — PyBullet visualization
    of three planned trajectories using subgroup planners so the
    relative-base joints stay pinned at HOME (verified with a
    runtime ``_assert_base_pinned`` guard, max drift 0).

New planning subgroups in bimanual_franka{,_soft}.py:
  • ``bimanual_fr3{,_soft}_left_gripper``  (2 DOF)
  • ``bimanual_fr3{,_soft}_right_gripper`` (2 DOF)
  • ``bimanual_fr3{,_soft}_dual_gripper``  (4 DOF)

Tests updated for the new dimensions; full suite passes (137 + 1
pre-existing flaky-CI skip).

Co-Authored-By: Claude Opus 4.7 (1M context) <noreply@anthropic.com>

File: assets/bimanual_fr3_description/urdf/bimanual_fr3.urdf (robot description, URDF)
Before this commit: robot bimanual_fr3, 30 links, 29 joints
Joints:
- joint fr3_left_finger_joint1: axis (none) -> 0 1 0; limit (none) -> lower=0.0 upper=0.04 effort=100 velocity=0.2; type fixed -> prismatic
- joint fr3_left_finger_joint2: axis (none) -> 0 1 0; limit (none) -> lower=0.0 upper=0.04 effort=100 velocity=0.2; mimic (none) -> joint=fr3_left_finger_joint1; type fixed -> prismatic
- joint fr3_right_finger_joint1: axis (none) -> 0 1 0; limit (none) -> lower=0.0 upper=0.04 effort=100 velocity=0.2; type fixed -> prismatic
- joint fr3_right_finger_joint2: axis (none) -> 0 1 0; limit (none) -> lower=0.0 upper=0.04 effort=100 velocity=0.2; mimic (none) -> joint=fr3_right_finger_joint1; type fixed -> prismatic

File: assets/bimanual_fr3_description/urdf/bimanual_fr3_soft.urdf (robot description, URDF)
Before this commit: robot bimanual_fr3_soft, 30 links, 29 joints
Joints:
- joint fr3_left_finger_joint1: axis (none) -> 0 1 0; limit (none) -> lower=0.0 upper=0.04 effort=100 velocity=0.2; origin xyz=0 0.025 0.0584 rpy=0 0 0 -> xyz=0 0 0.0584 rpy=0 0 0; type fixed -> prismatic
- joint fr3_left_finger_joint2: axis (none) -> 0 1 0; limit (none) -> lower=0.0 upper=0.04 effort=100 velocity=0.2; mimic (none) -> joint=fr3_left_finger_joint1; origin xyz=0 -0.025 0.0584 rpy=0 0 3.141592653589793 -> xyz=0 0 0.0584 rpy=0 0 3.141592653589793; type fixed -> prismatic
- joint fr3_right_finger_joint1: axis (none) -> 0 1 0; limit (none) -> lower=0.0 upper=0.04 effort=100 velocity=0.2; origin xyz=0 0.025 0.0584 rpy=0 0 0 -> xyz=0 0 0.0584 rpy=0 0 0; type fixed -> prismatic
- joint fr3_right_finger_joint2: axis (none) -> 0 1 0; limit (none) -> lower=0.0 upper=0.04 effort=100 velocity=0.2; mimic (none) -> joint=fr3_right_finger_joint1; origin xyz=0 -0.025 0.0584 rpy=0 0 3.141592653589793 -> xyz=0 0 0.0584 rpy=0 0 3.141592653589793; type fixed -> prismatic

File: bimanual_franka_planning/resources/robot/bimanual_fr3/bimanual_fr3_spherized.urdf (robot description, URDF)
Before this commit: robot bimanual_fr3, 30 links, 29 joints
Joints:
- joint fr3_left_finger_joint1: axis (none) -> 0 1 0; limit (none) -> lower=0.0 upper=0.04 effort=100 velocity=0.2; type fixed -> prismatic
- joint fr3_left_finger_joint2: axis (none) -> 0 1 0; limit (none) -> lower=0.0 upper=0.04 effort=100 velocity=0.2; mimic (none) -> joint=fr3_left_finger_joint1; type fixed -> prismatic
- joint fr3_right_finger_joint1: axis (none) -> 0 1 0; limit (none) -> lower=0.0 upper=0.04 effort=100 velocity=0.2; type fixed -> prismatic
- joint fr3_right_finger_joint2: axis (none) -> 0 1 0; limit (none) -> lower=0.0 upper=0.04 effort=100 velocity=0.2; mimic (none) -> joint=fr3_right_finger_joint1; type fixed -> prismatic

File: bimanual_franka_planning/resources/robot/bimanual_fr3/bimanual_fr3_viz.urdf (robot description, URDF)
Before this commit: robot bimanual_fr3, 30 links, 29 joints
Joints:
- joint fr3_left_finger_joint1: axis (none) -> 0 1 0; limit (none) -> lower=0.0 upper=0.04 effort=100 velocity=0.2; type fixed -> prismatic
- joint fr3_left_finger_joint2: axis (none) -> 0 1 0; limit (none) -> lower=0.0 upper=0.04 effort=100 velocity=0.2; mimic (none) -> joint=fr3_left_finger_joint1; type fixed -> prismatic
- joint fr3_right_finger_joint1: axis (none) -> 0 1 0; limit (none) -> lower=0.0 upper=0.04 effort=100 velocity=0.2; type fixed -> prismatic
- joint fr3_right_finger_joint2: axis (none) -> 0 1 0; limit (none) -> lower=0.0 upper=0.04 effort=100 velocity=0.2; mimic (none) -> joint=fr3_right_finger_joint1; type fixed -> prismatic

File: bimanual_franka_planning/resources/robot/bimanual_fr3_soft/bimanual_fr3_soft_spherized.urdf (robot description, URDF)
Before this commit: robot bimanual_fr3_soft, 30 links, 29 joints
Joints:
- joint fr3_left_finger_joint1: axis (none) -> 0 1 0; limit (none) -> lower=0.0 upper=0.04 effort=100 velocity=0.2; origin xyz=0 0.025 0.0584 rpy=0 0 0 -> xyz=0 0 0.0584 rpy=0 0 0; type fixed -> prismatic
- joint fr3_left_finger_joint2: axis (none) -> 0 1 0; limit (none) -> lower=0.0 upper=0.04 effort=100 velocity=0.2; mimic (none) -> joint=fr3_left_finger_joint1; origin xyz=0 -0.025 0.0584 rpy=0 0 3.141592653589793 -> xyz=0 0 0.0584 rpy=0 0 3.141592653589793; type fixed -> prismatic
- joint fr3_right_finger_joint1: axis (none) -> 0 1 0; limit (none) -> lower=0.0 upper=0.04 effort=100 velocity=0.2; origin xyz=0 0.025 0.0584 rpy=0 0 0 -> xyz=0 0 0.0584 rpy=0 0 0; type fixed -> prismatic
- joint fr3_right_finger_joint2: axis (none) -> 0 1 0; limit (none) -> lower=0.0 upper=0.04 effort=100 velocity=0.2; mimic (none) -> joint=fr3_right_finger_joint1; origin xyz=0 -0.025 0.0584 rpy=0 0 3.141592653589793 -> xyz=0 0 0.0584 rpy=0 0 3.141592653589793; type fixed -> prismatic

File: bimanual_franka_planning/resources/robot/bimanual_fr3_soft/bimanual_fr3_soft_viz.urdf (robot description, URDF)
Before this commit: robot bimanual_fr3_soft, 30 links, 29 joints
Joints:
- joint fr3_left_finger_joint1: axis (none) -> 0 1 0; limit (none) -> lower=0.0 upper=0.04 effort=100 velocity=0.2; origin xyz=0 0.025 0.0584 rpy=0 0 0 -> xyz=0 0 0.0584 rpy=0 0 0; type fixed -> prismatic
- joint fr3_left_finger_joint2: axis (none) -> 0 1 0; limit (none) -> lower=0.0 upper=0.04 effort=100 velocity=0.2; mimic (none) -> joint=fr3_left_finger_joint1; origin xyz=0 -0.025 0.0584 rpy=0 0 3.141592653589793 -> xyz=0 0 0.0584 rpy=0 0 3.141592653589793; type fixed -> prismatic
- joint fr3_right_finger_joint1: axis (none) -> 0 1 0; limit (none) -> lower=0.0 upper=0.04 effort=100 velocity=0.2; origin xyz=0 0.025 0.0584 rpy=0 0 0 -> xyz=0 0 0.0584 rpy=0 0 0; type fixed -> prismatic
- joint fr3_right_finger_joint2: axis (none) -> 0 1 0; limit (none) -> lower=0.0 upper=0.04 effort=100 velocity=0.2; mimic (none) -> joint=fr3_right_finger_joint1; origin xyz=0 -0.025 0.0584 rpy=0 0 3.141592653589793 -> xyz=0 0 0.0584 rpy=0 0 3.141592653589793; type fixed -> prismatic

File: bimanual_franka_planning/resources/robot/single_fr3/single_fr3.urdf (robot description, URDF)
Before this commit: robot fr3, 14 links, 13 joints
Joints:
- joint fr3_finger_joint1: type fixed -> prismatic
- joint fr3_finger_joint2: type fixed -> prismatic

File: bimanual_franka_planning/resources/robot/single_fr3/single_fr3_spherized.urdf (robot description, URDF)
Before this commit: robot fr3, 14 links, 13 joints
Joints:
- joint fr3_finger_joint1: type fixed -> prismatic
- joint fr3_finger_joint2: type fixed -> prismatic

File: bimanual_franka_planning/resources/robot/single_fr3_soft/single_fr3_soft.urdf (robot description, URDF)
Before this commit: robot fr3_soft, 14 links, 13 joints
Joints:
- joint fr3_finger_joint1: axis (none) -> 0 1 0; limit (none) -> lower=0.0 upper=0.04 effort=100 velocity=0.2; origin xyz=0 0.025 0.0584 rpy=0 0 0 -> xyz=0 0 0.0584 rpy=0 0 0; type fixed -> prismatic
- joint fr3_finger_joint2: axis (none) -> 0 1 0; limit (none) -> lower=0.0 upper=0.04 effort=100 velocity=0.2; mimic (none) -> joint=fr3_finger_joint1; origin xyz=0 -0.025 0.0584 rpy=0 0 3.141592653589793 -> xyz=0 0 0.0584 rpy=0 0 3.141592653589793; type fixed -> prismatic

File: bimanual_franka_planning/resources/robot/single_fr3_soft/single_fr3_soft_spherized.urdf (robot description, URDF)
Before this commit: robot fr3_soft, 14 links, 13 joints
Joints:
- joint fr3_finger_joint1: axis (none) -> 0 1 0; limit (none) -> lower=0.0 upper=0.04 effort=100 velocity=0.2; origin xyz=0 0.025 0.0584 rpy=0 0 0 -> xyz=0 0 0.0584 rpy=0 0 0; type fixed -> prismatic
- joint fr3_finger_joint2: axis (none) -> 0 1 0; limit (none) -> lower=0.0 upper=0.04 effort=100 velocity=0.2; mimic (none) -> joint=fr3_finger_joint1; origin xyz=0 -0.025 0.0584 rpy=0 0 3.141592653589793 -> xyz=0 0 0.0584 rpy=0 0 3.141592653589793; type fixed -> prismatic
