Commit message: Model UMI wsg50-Franka finger holder on soft FR3 URDFs
Adds the printed finger-holder adapter that sits between the WSG slider
and the soft finger to the URDF generator and regenerated artifacts:

* New canonical mesh sources at planning root: finger_holder_{left,right}.stl
  (mirrored pair from the UMI wsg50-Franka mount assembly, in metres).
* tools/build_soft_fr3_urdfs.py stages the holder STLs into each soft
  resource tree and stamps a second <visual>+<collision> on each finger
  link with the per-side rotation that aligns the STL extension axis
  (STL -Y, 70 mm) with the link finger axis (link +Z) and the STL X
  cross with the link gripping pad (link Y).  Holder occupies link
  Z [5, 75] mm, overlapping the inner half of the soft finger.
* Soft finger shifted +20 mm along link +Z so it seats on the holder's
  outer face — the kinematic "1-2 cm longer gripper" the real hardware
  exhibits.  Sphere envelope and hand_tcp origin both bumped to match.
* Holder sphere collision (4 spheres, r=0.028) added for FK gen.
* Regenerated single + bimanual URDFs (mesh/spherized/viz), the
  assets/ mirror, and all four cricket FK headers.  Python interface
  is unchanged: fr3_*_link8 and joint names referenced by
  single_franka_soft.py / bimanual_franka_soft.py are preserved.

Co-Authored-By: Claude Opus 4.7 (1M context) <noreply@anthropic.com>

File: assets/bimanual_fr3_description/urdf/bimanual_fr3_soft.urdf (robot description, URDF)
Before this commit: robot bimanual_fr3_soft, 30 links, 29 joints
Links:
- link fr3_left_leftfinger: geometry collision mesh filename=package://meshes/robot_ee/franka_hand_soft/collision/finger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; collision mesh filename=package://meshes/robot_ee/franka_hand_soft/collision/finger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
- link fr3_left_rightfinger: geometry collision mesh filename=package://meshes/robot_ee/franka_hand_soft/collision/finger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; collision mesh filename=package://meshes/robot_ee/franka_hand_soft/collision/finger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
- link fr3_right_leftfinger: geometry collision mesh filename=package://meshes/robot_ee/franka_hand_soft/collision/finger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; collision mesh filename=package://meshes/robot_ee/franka_hand_soft/collision/finger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
- link fr3_right_rightfinger: geometry collision mesh filename=package://meshes/robot_ee/franka_hand_soft/collision/finger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; collision mesh filename=package://meshes/robot_ee/franka_hand_soft/collision/finger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
Joints:
- joint fr3_left_hand_tcp_joint: origin xyz=0 0 0.1034 rpy=0 0 0 -> xyz=0 0 0.12340000000000001 rpy=0 0 0
- joint fr3_right_hand_tcp_joint: origin xyz=0 0 0.1034 rpy=0 0 0 -> xyz=0 0 0.12340000000000001 rpy=0 0 0

File: bimanual_franka_planning/resources/robot/bimanual_fr3_soft/bimanual_fr3_soft_spherized.urdf (robot description, URDF)
Before this commit: robot bimanual_fr3_soft, 30 links, 29 joints
Links:
- link fr3_left_leftfinger: geometry collision sphere radius=0.02; collision sphere radius=0.024
- link fr3_left_rightfinger: geometry collision sphere radius=0.02; collision sphere radius=0.024
- link fr3_right_leftfinger: geometry collision sphere radius=0.02; collision sphere radius=0.024
- link fr3_right_rightfinger: geometry collision sphere radius=0.02; collision sphere radius=0.024
Joints:
- joint fr3_left_hand_tcp_joint: origin xyz=0 0 0.1034 rpy=0 0 0 -> xyz=0 0 0.12340000000000001 rpy=0 0 0
- joint fr3_right_hand_tcp_joint: origin xyz=0 0 0.1034 rpy=0 0 0 -> xyz=0 0 0.12340000000000001 rpy=0 0 0

File: bimanual_franka_planning/resources/robot/bimanual_fr3_soft/bimanual_fr3_soft_viz.urdf (robot description, URDF)
Before this commit: robot bimanual_fr3_soft, 30 links, 29 joints
Links:
- link fr3_left_leftfinger: geometry visual mesh filename=package://meshes/robot_ee/franka_hand_soft/visual/finger.stl; visual mesh filename=package://meshes/robot_ee/franka_hand_soft/visual/finger_ho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
- link fr3_left_rightfinger: geometry visual mesh filename=package://meshes/robot_ee/franka_hand_soft/visual/finger.stl; visual mesh filename=package://meshes/robot_ee/franka_hand_soft/visual/finger_ho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
- link fr3_right_leftfinger: geometry visual mesh filename=package://meshes/robot_ee/franka_hand_soft/visual/finger.stl; visual mesh filename=package://meshes/robot_ee/franka_hand_soft/visual/finger_ho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
- link fr3_right_rightfinger: geometry visual mesh filename=package://meshes/robot_ee/franka_hand_soft/visual/finger.stl; visual mesh filename=package://meshes/robot_ee/franka_hand_soft/visual/finger_ho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
Joints:
- joint fr3_left_hand_tcp_joint: origin xyz=0 0 0.1034 rpy=0 0 0 -> xyz=0 0 0.12340000000000001 rpy=0 0 0
- joint fr3_right_hand_tcp_joint: origin xyz=0 0 0.1034 rpy=0 0 0 -> xyz=0 0 0.12340000000000001 rpy=0 0 0

File: bimanual_franka_planning/resources/robot/single_fr3_soft/single_fr3_soft.urdf (robot description, URDF)
Before this commit: robot fr3_soft, 14 links, 13 joints
Links:
- link fr3_leftfinger: geometry collision mesh filename=package://meshes/robot_ee/franka_hand_soft/collision/finger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; collision mesh filename=package://meshes/robot_ee/franka_hand_soft/collision/finger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
- link fr3_rightfinger: geometry collision mesh filename=package://meshes/robot_ee/franka_hand_soft/collision/finger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; collision mesh filename=package://meshes/robot_ee/franka_hand_soft/collision/finger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
Joints:
- joint fr3_hand_tcp_joint: origin xyz=0 0 0.1034 rpy=0 0 0 -> xyz=0 0 0.12340000000000001 rpy=0 0 0

File: bimanual_franka_planning/resources/robot/single_fr3_soft/single_fr3_soft_spherized.urdf (robot description, URDF)
Before this commit: robot fr3_soft, 14 links, 13 joints
Links:
- link fr3_leftfinger: geometry collision sphere radius=0.02; collision sphere radius=0.024
- link fr3_rightfinger: geometry collision sphere radius=0.02; collision sphere radius=0.024
Joints:
- joint fr3_hand_tcp_joint: origin xyz=0 0 0.1034 rpy=0 0 0 -> xyz=0 0 0.12340000000000001 rpy=0 0 0
